Commit message: tried to fix the slam

File: src/nexus_description/urdf/nexus_4wd_mecanum.urdf.xacro (robot description, xacro)
@@ -331,4 +331,19 @@
     </visual>
   </link>
+   <!-- LiDAR -->
+  <joint name="laser_joint" type="fixed">
+    <origin xyz="0.205 0 0.15" rpy="0 0 0" />
+    <parent link="base_link"/>
+    <child link="laser"/>
+  </joint>
+  <link name="laser">
+    <visual>
+      <origin xyz="0 0 0" rpy="0 0 0" />
+      <geometry>
+        <cylinder radius="0.035" length="0.05"/>
+      </geometry>
+      <material name="black"/>
+    </visual>
+  </link>
   <!--
   <xacro:include filename="$(ros2 pkg prefix nexus_description)/urdf/nexus_4wd_mecanum.gazebo"/>
